Commit message: Changed way actions are being called, move_robot_client and move_ball_client not needed anymore. Also added frontal mass to the urdf model

File: urdf/ex3_arm.xacro (robot description, xacro)
@@ -90,5 +90,5 @@
   <link name="arm_base_link">
   	<inertial>
-  		<mass value="0.1"/>
+  		<mass value="0.5"/>
   		<origin xyz="0 0 0" rpy="0 0 0" />
   		<inertia ixx="0.0000416666667" ixy="0" ixz="0" iyy="0.0000416666667" iyz="0" izz="0.0000416666667"/>
